File: hardware/PicoLink.kicad_pcb (KiCad board)
At the start: 2 copper layers, 53.2 x 24.8 mm, 50 parts, among them J1 USB_C_Receptacle_GCT_USB4110-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, J3 Conn_ARM_JTAG_SWD_10, J5 Conn_01x03, J6 Conn_01x03, SW1 434123025826_BTN, U1 W25Q16JV, U2 RP2040, U3 SWD_JTAG_10pin, U4 W25Q32JVSS, U5 AP2112K-3.3, U6 AMS1117-3.3, Y1 CSTNE12M0GH5L000R0

Commit message: [07-16-2030] finish rough routing
Parts:
- removed C10, C11, C12, C13, C3, C4, C5, C6, C7, C8: 0.1u, Capacitor_SMD:C_0603_1608Metric
- removed C14, C15: 22u, McuOnEclipse:C_0805
- removed C2, C9: 2u2, Capacitor_SMD:C_0603_1608Metric
- removed D1: red, McuOnEclipse:LED_0603
- removed D5: green, McuOnEclipse:LED_0603
- removed H1: Logo HSLU, McuOnEclipse:Hochschule_Luzern_New
- removed H2: QR, McuOnEclipse:QR_McuOnEclipse_Silkscreen
- removed J1: USB_C_Receptacle_GCT_USB4110-GF-A, McuOnEclipse:USB_C_Receptacle_GCT_USB4110-GF-A
- removed J5, J6: Conn_01x03, Connector_PinHeader_2.54mm:PinHeader_1x03_P2.54mm_Vertical
- removed R10, R11, R15, R16, R9: 100, Resistor_SMD:R_0603_1608Metric
- removed R18, R7, R8: 2k2, Resistor_SMD:R_0603_1608Metric
- removed R2, R5: 5k1, Resistor_SMD:R_0603_1608Metric
- removed R3, R4: 27, Resistor_SMD:R_0603_1608Metric
- removed RP2040: RP2040, McuOnEclipse:QFN-56-1EP_7x7mm_P0.4mm_EP3.2x3.2mm
- removed SW1: 434123025826_BTN, McuOnEclipse:434123025826_BTN
- removed U1: W25Q16JV, McuOnEclipse:USON_2x3x0.6mm
- removed U2: RP2040, Package_DFN_QFN:QFN-56-1EP_7x7mm_P0.4mm_EP5.6x5.6mm
- removed U3: SWD_JTAG_10pin, McuOnEclipse:SWD_Pin_Header_Straight_2x05_Pitch1.27mm_SMD
- removed U5: AP2112K-3.3, McuOnEclipse:IC-SOT25
- removed Y1: CSTNE12M0GH5L000R0, McuOnEclipse:Resonator_SMD_Murata_CSTxExxV-3Pin_3.0x1.1mm
- added C1: 12pF, Capacitor_SMD:C_0603_1608Metric_Pad1.08x0.95mm_HandSolder, F.Cu at (155.6, 99.8)
- added C16: 100nF, Capacitor_SMD:C_0603_1608Metric_Pad1.08x0.95mm_HandSolder, F.Cu at (152.4, 78.6)
- added C17: 22uF, Capacitor_SMD:C_0603_1608Metric_Pad1.08x0.95mm_HandSolder, F.Cu at (158.3, 77.5)
- added C18: 22uF, Capacitor_SMD:C_0603_1608Metric_Pad1.08x0.95mm_HandSolder, F.Cu at (168.9, 80.9)
- added C19: 100nF, Capacitor_SMD:C_0603_1608Metric_Pad1.08x0.95mm_HandSolder, F.Cu at (158.8, 85.6)
- added C20: 2u2F, Capacitor_SMD:C_0603_1608Metric_Pad1.08x0.95mm_HandSolder, F.Cu at (152.4, 73.4)
- added C21: 100nF, Capacitor_SMD:C_0603_1608Metric_Pad1.08x0.95mm_HandSolder, F.Cu at (152.4, 76.9)
- added C22: 100nF, Capacitor_SMD:C_0603_1608Metric_Pad1.08x0.95mm_HandSolder, F.Cu at (152.4, 75.2)
- added C23: 12pF, Capacitor_SMD:C_0603_1608Metric_Pad1.08x0.95mm_HandSolder, F.Cu at (155.6, 98.2)
- added C26: 2u2F, Capacitor_SMD:C_0603_1608Metric_Pad1.08x0.95mm_HandSolder, F.Cu at (160.5, 85.6)
- added C27: 100nF, Capacitor_SMD:C_0603_1608Metric_Pad1.08x0.95mm_HandSolder, F.Cu at (168.8, 85.6)
- added C28: 100nF, Capacitor_SMD:C_0603_1608Metric_Pad1.08x0.95mm_HandSolder, F.Cu at (170.5, 85.6)
- added C29: 100nF, Capacitor_SMD:C_0603_1608Metric_Pad1.08x0.95mm_HandSolder, F.Cu at (162.2, 85.6)
- added C30: 100nF, Capacitor_SMD:C_0603_1608Metric_Pad1.08x0.95mm_HandSolder, F.Cu at (163.8, 85.6)
- added C31: 100nF, Capacitor_SMD:C_0603_1608Metric_Pad1.08x0.95mm_HandSolder, F.Cu at (165.4, 85.6)
- added C32: 100nF, Capacitor_SMD:C_0603_1608Metric_Pad1.08x0.95mm_HandSolder, F.Cu at (167.2, 85.6)
- added D2: green, LED_SMD:LED_0805_2012Metric_Pad1.15x1.40mm_HandSolder, F.Cu at (167.8, 97.5)
- added D3: red, LED_SMD:LED_0805_2012Metric_Pad1.15x1.40mm_HandSolder, F.Cu at (157.2, 73.8)
- added J2: USB_C_Receptacle_USB2.0_14P, Connector_USB:USB_C_Receptacle_GCT_USB4110, F.Cu at (176.5, 94.0)
- added J4: TARGET, Connector_PinHeader_2.54mm:PinHeader_1x03_P2.54mm_Vertical, B.Cu at (138.2, 88.7)
- added J7: UART, Connector_PinHeader_2.54mm:PinHeader_1x03_P2.54mm_Vertical, B.Cu at (142.8, 88.6)
- added J8: SIGROK_INPUT, Connector_PinHeader_2.54mm:PinHeader_1x07_P2.54mm_Horizontal, B.Cu at (148.4, 107.6)
- added J9: SIGROK_ADC, Connector_PinHeader_2.54mm:PinHeader_1x03_P2.54mm_Vertical, B.Cu at (163.0, 97.1)
- added R1: 5K1, Resistor_SMD:R_0805_2012Metric_Pad1.20x1.40mm_HandSolder, F.Cu at (167.8, 95.2)
- added R12: 27, Resistor_SMD:R_0805_2012Metric_Pad1.20x1.40mm_HandSolder, F.Cu at (167.7, 93.1)
- added R13: 27, Resistor_SMD:R_0805_2012Metric_Pad1.20x1.40mm_HandSolder, F.Cu at (167.7, 90.9)
- added R14: 100, Resistor_SMD:R_0805_2012Metric_Pad1.20x1.40mm_HandSolder, F.Cu at (137.2, 100.8)
- added R17: 100, Resistor_SMD:R_0805_2012Metric_Pad1.20x1.40mm_HandSolder, F.Cu at (137.2, 102.9)
- added R19: 100, Resistor_SMD:R_0805_2012Metric_Pad1.20x1.40mm_HandSolder, F.Cu at (137.2, 105.0)
- added R20: 2K2, Resistor_SMD:R_0805_2012Metric_Pad1.20x1.40mm_HandSolder, F.Cu at (146.4, 76.4)
- added R21: 1K, Resistor_SMD:R_0805_2012Metric_Pad1.20x1.40mm_HandSolder, F.Cu at (167.8, 99.5)
- added R22: 1K, Resistor_SMD:R_0805_2012Metric_Pad1.20x1.40mm_HandSolder, F.Cu at (155.8, 77.4)
- added R23: 100, Resistor_SMD:R_0805_2012Metric_Pad1.20x1.40mm_HandSolder, F.Cu at (147.8, 89.2)
- added R24: 100, Resistor_SMD:R_0805_2012Metric_Pad1.20x1.40mm_HandSolder, F.Cu at (147.8, 91.3)
- added R25: 100, Resistor_SMD:R_0805_2012Metric_Pad1.20x1.40mm_HandSolder, F.Cu at (147.8, 93.3)
- added R26: 100, Resistor_SMD:R_0805_2012Metric_Pad1.20x1.40mm_HandSolder, F.Cu at (147.8, 95.5)
- added R6: 5K1, Resistor_SMD:R_0805_2012Metric_Pad1.20x1.40mm_HandSolder, F.Cu at (167.7, 88.9)
- added RP1: RP2040, Package_DFN_QFN:QFN-56-1EP_7x7mm_P0.4mm_EP3.2x3.2mm, F.Cu at (155.7, 92.7)
- added SW2: BOOT SELECTOR, Button_Switch_SMD:SW_Push_1P1T_NO_6x6mm_H9.5mm, F.Cu at (139.8, 83.0)
- added Y2: 12Mhz HC49-SD, Crystal:Crystal_SMD_HC49-SD_HandSoldering, F.Cu at (156.3, 102.6)
- J3: value Conn_ARM_JTAG_SWD_10 -> ARM_JTAG_10Pin; footprint Connector_PinHeader_1.27mm:PinHeader_2x05_P1.27mm_Vertical_SMD -> Connector_IDC:IDC-Header_2x05_P2.54mm_Vertical; moved to B.Cu
- U4: value W25Q32JVSS -> W25Q16JVSS
- moved FID2 94.4 mm to (174.8, 84.5)
- moved H5 51.8 mm to (176.2, 79.0)
- moved H6 50.6 mm to (127.3, 79.0)
- moved H3 45.6 mm to (175.9, 108.0)
- moved H4 44.1 mm to (127.0, 108.2)
- moved FID1 38.5 mm to (170.2, 103.2)
- moved FID3 27.0 mm to (141.1, 100.5)
- moved U6 27.0 mm to (163.5, 78.5), turned to 90 degrees
- moved U4 17.6 mm to (152.7, 82.9)
- moved J3 4.20 mm to (128.0, 88.4), turned to 180 degrees
Connections:
- J3 pad 1: unconnected-(J3-VTref-Pad1) -> +3.3V
- J3 pad 10: unconnected-(J3-~{RESET}-Pad10) -> Net-(J3-~{RESET})
- J3 pad 2: unconnected-(J3-SWDIO/TMS-Pad2) -> Net-(J3-SWDIO/TMS)
- J3 pad 3: Net-(J3-GND-Pad3) -> GND
- J3 pad 4: unconnected-(J3-SWCLK/TCK-Pad4) -> Net-(J3-SWCLK/TCK)
- J3 pad 5: Net-(J3-GND-Pad3) -> GND
- J3 pad 9: unconnected-(J3-GNDDetect-Pad9) -> GND
- U4 pad 1: unconnected-(U4-~{CS}-Pad1) -> /SPI_SS_N
- U4 pad 2: unconnected-(U4-DO(IO1)-Pad2) -> /SPI_SD1
- U4 pad 3: unconnected-(U4-IO2-Pad3) -> /SPI_SD2
- U4 pad 4: unconnected-(U4-GND-Pad4) -> GND
- U4 pad 5: unconnected-(U4-DI(IO0)-Pad5) -> /SPI_SD0
- U4 pad 6: unconnected-(U4-CLK-Pad6) -> /SPI_SCLK
- U4 pad 7: unconnected-(U4-IO3-Pad7) -> /SPI_SD3
- U4 pad 8: unconnected-(U4-VCC-Pad8) -> +3.3V
- U6 pad 1: unconnected-(U6-GND-Pad1) -> GND
- U6 pad 2: unconnected-(U6-VO-Pad2) -> +3.3V
- U6 pad 3: unconnected-(U6-VI-Pad3) -> +5V
Routing:
- net GND: track 24.7 -> 245.7 mm, vias 68 -> 0
- net SWD_DIO: track 43.1 -> 0.00 mm, vias 10 -> 0
- net /SIGROK_IN7: track 0.00 -> 41.4 mm, vias 0 -> 2
- net SWD_CLK: track 40.3 -> 0.00 mm, vias 8 -> 0
- net TGT_SWDIO: track 14.5 -> 54.8 mm
- net TGT_SWCLK: track 15.2 -> 48.9 mm
- net /SIGROK_IN6: track 0.00 -> 33.5 mm
- net /SIGROK_IN5: track 0.00 -> 31.6 mm
- net /SIGROK_IN4: track 0.00 -> 29.7 mm
- net Net-(J3-SWDIO/TMS): track 0.00 -> 28.3 mm
- net /SIGROK_IN3: track 0.00 -> 27.6 mm
- net /SIGROK_IN2: track 0.00 -> 25.5 mm
- net /SIGROK_IN1: track 0.00 -> 24.3 mm
- net Net-(J3-SWCLK/TCK): track 0.00 -> 23.7 mm
- net Net-(J5-Pin_1): track 22.5 -> 0.00 mm
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- removed copper zone on B.Cu, net GND
- removed copper zone on F.Cu, net GND
Other:
- board outline removed
- board text removed: "Boot Sel"
- board text removed: "CLK"
- board text removed: "DIO"
- board text removed: "GND"
- board text removed: "RP2040"
- board text removed: "Rx"
- board text removed: "Tx"
- board text removed: "UART"

Commit message: [07-17-1304] add edge cut
Update README.md
Parts:
- J8: footprint Connector_PinHeader_2.54mm:PinHeader_1x07_P2.54mm_Horizontal -> Connector_PinHeader_2.54mm:PinHeader_1x07_P2.54mm_Vertical
- moved FID3 12.6 mm to (135.1, 89.5)
- moved FID2 11.2 mm to (164.4, 88.7)
- moved C20 6.09 mm to (148.5, 78.0), turned to -90 degrees
- moved D3 4.66 mm to (159.6, 77.8), turned to -90 degrees
- moved R17 3.98 mm to (140.7, 101.0)
- moved R19 3.98 mm to (140.7, 103.0)
- moved R14 3.98 mm to (140.7, 98.9)
- moved J3 3.94 mm to (131.9, 88.9)
- moved H4 3.71 mm to (130.7, 107.9)
- moved C22 3.63 mm to (150.2, 78.0), turned to -90 degrees
- moved H6 3.47 mm to (130.7, 79.9)
- moved H5 2.98 mm to (176.7, 82.0)
- moved R20 2.45 mm to (146.4, 78.9), turned to 90 degrees
- moved H3 2.00 mm to (175.4, 106.1)
- moved J4 1.98 mm to (139.8, 89.8)
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Routing:
- net +3.3V: track 126.1 -> 115.5 mm
- net /SPI_SS_N: track 21.4 -> 15.8 mm
- net TGT_RESET: track 19.8 -> 14.8 mm
- net GND: track 245.7 -> 242.1 mm
- net Net-(J4-Pin_1): track 11.1 -> 8.03 mm
- net Net-(J4-Pin_3): track 16.2 -> 13.2 mm
- net Net-(D3-K): track 2.68 -> 5.00 mm
- net TGT_SWDIO: track 54.8 -> 52.8 mm
- net /SPI_SD1: track 14.7 -> 12.9 mm
- net /SPI_SD2: track 13.2 -> 11.3 mm
- net Net-(J7-Pin_1): track 6.44 -> 4.85 mm
- net Net-(J7-Pin_3): track 4.83 -> 3.30 mm
- net /SIGROK_IN2: track 25.5 -> 24.0 mm
- net /SIGROK_IN3: track 27.6 -> 26.1 mm
- net /SIGROK_IN1: track 24.3 -> 22.8 mm
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- added copper zone on F.Cu, net +3.3V
Other:
- board outline added: 56.1 x 38.2 mm
- board text added: "PIKO"

Commit message: [07-17-1556] update silkscreen
Parts:
- added REF**: OSHW-Logo2_7.3x6mm_SilkScreen, Symbol:OSHW-Logo2_7.3x6mm_SilkScreen, F.Cu at (169.8, 108.2)
- moved FID3 13.3 mm to (136.8, 76.3)
- moved FID2 12.7 mm to (176.0, 83.5)
- moved H5 2.87 mm to (176.3, 79.2)
- moved H3 1.73 mm to (176.1, 107.7)
- moved H6 0.89 mm to (130.1, 79.2)
- moved H4 0.20 mm to (130.5, 107.9)
Routing:
- net GND: track 242.1 -> 244.6 mm
- net Net-(J4-Pin_1): track 8.03 -> 10.4 mm
- net Net-(J4-Pin_3): track 13.2 -> 14.4 mm
- net Net-(J7-Pin_1): track 4.85 -> 5.99 mm
Other:
- board text removed: "PicoDAP V0.2 Erich Styger 31-Mar-2023"

Commit message: [07-18-2108] add svg schematic
Parts:
- removed REF**: OSHW-Logo2_7.3x6mm_SilkScreen, Symbol:OSHW-Logo2_7.3x6mm_SilkScreen
- moved C20 34.6 mm to (169.4, 105.5), turned to 0 degrees
- moved C22 32.1 mm to (169.4, 103.8), turned to 0 degrees
- moved C21 29.7 mm to (169.4, 102.0), turned to 0 degrees
- moved FID1 6.01 mm to (169.1, 109.1)
Connections:
- C20 pad 1: +3.3V -> Net-(RP1-VREG_VOUT)
- C21 pad 1: +3.3V -> Net-(RP1-VREG_VOUT)
- C22 pad 1: +3.3V -> Net-(RP1-VREG_VOUT)
- RP1 pad 23: +3.3V -> Net-(RP1-VREG_VOUT)
- RP1 pad 45: +3.3V -> Net-(RP1-VREG_VOUT)
- RP1 pad 50: +3.3V -> Net-(RP1-VREG_VOUT)
Routing:
- net Net-(RP1-VREG_VOUT): track 0.00 -> 34.0 mm
- net +3.3V: track 115.5 -> 142.2 mm, vias 2 -> 6
- net GND: track 244.6 -> 250.8 mm
- net /USB_DM: track 12.2 -> 14.9 mm
- net +5V: track 33.6 -> 36.1 mm
- net unconnected-(RP1-GPIO0-Pad2): track 0.00 -> 1.46 mm
- net /SWDIR: track 0.00 -> 1.46 mm
- net /USB_DP: track 12.2 -> 13.4 mm
- net /SPI_SD3: track 9.75 -> 11.0 mm
- net unconnected-(RP1-GPIO9-Pad12): track 0.00 -> 1.16 mm
- net unconnected-(RP1-GPIO8-Pad11): track 0.00 -> 1.16 mm
- net unconnected-(RP1-GPIO7-Pad9): track 0.00 -> 1.16 mm
- net /SPI_SS_N: track 15.8 -> 16.8 mm
- net /SPI_SCLK: track 8.14 -> 9.12 mm
- net unconnected-(RP1-GPIO21-Pad32): track 0.00 -> 0.96 mm
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